Commit message: Ajout de log pour le calcul de position 3D à partir des angles

File: src/robotic_arm/model/model.xacro (robot description, xacro)
@@ -5,5 +5,5 @@
         <link name="base_link">
                 <inertial>
-                        <mass value="40"/>
+                        <mass value="1500"/>
                         <inertia ixx="0.1" ixy="0.0" ixz="0.0" iyy="0.1" iyz="0" izz="0.1" />
                 </inertial>
@@ -44,5 +44,5 @@
                 <child link="first_arm_link"/>
                 <axis xyz="0 0 1"/>
-                <limit lower="-1.571" upper="1.571" effort="100" velocity="10"/>
+                <limit lower="-1.571" upper="1.571" effort="1000" velocity="1"/>
         </joint>
         <link name="second_arm_link">
@@ -69,5 +69,5 @@
                 <child link="second_arm_link"/>
                 <axis xyz="0 1 0"/>
-                <limit lower="-1.571" upper="1.571" effort="100" velocity="10"/>
+                <limit lower="-1.571" upper="1.571" effort="1000" velocity="1"/>
         </joint>
         <link name="third_arm_link">
@@ -94,5 +94,5 @@
                 <child link="third_arm_link"/>
                 <axis xyz="0 1 0"/>
-                <limit lower="-1.571" upper="1.571" effort="100" velocity="10"/>
+                <limit lower="-1.571" upper="1.571" effort="1000" velocity="1"/>
         </joint>
         <link name="fourth_arm_link">
@@ -119,5 +119,25 @@
                 <child link="fourth_arm_link"/>
                 <axis xyz="0 1 0"/>
-                <limit lower="-1.571" upper="1.571" effort="100" velocity="10"/>
+                <limit lower="-1.571" upper="1.571" effort="1000" velocity="1"/>
+        </joint>
+        <link name="visual_reference">
+                <inertial>
+                        <mass value="1"/>
+                        <inertia ixx="0.001" ixy="0.0" ixz="0.0" iyy="0.001" iyz="0" izz="0.001"/>
+                </inertial>
+                <visual>
+                        <geometry>
+                                <box size="${arm_length} ${arm_width} ${0.2}"/>
+                        </geometry>
+                        <origin xyz="0 0 0" rpy="0 0 0"/>
+                        <material name="red">
+                                <color rgba="1 0 0 1"/>
+                        </material>
+                </visual>
+        </link>
+        <joint name="visual_reference_joint" type="fixed">
+                <origin xyz="0 0 ${arm_height - 0.3}" rpy="0 0 0"/>
+                <parent link="fourth_arm_link"/>
+                <child link="visual_reference"/>
         </joint>
         <ros2_control name="RobotController" type="system">
